File: Hardware/MoodBadge.brd (EAGLE design)
At the start: 54 x 94.8 mm, 46 parts

Commit message: updates
Parts:
- renumbered U$7 to XTAL
Changed lines of the file:
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@@
 <attribute name="VALUE" x="23.7744" y="51.3842" size="1.27" layer="28" rot="MR90"/>
 </element>
-<element name="U$7" library="OrlandoRonMod" package="CA-301" value="CRYSTAL-CA-310" x="32.3596" y="39.2176" smashed="yes" rot="R90">
+<element name="XTAL" library="OrlandoRonMod" package="CA-301" value="CRYSTAL-CA-310" x="32.3596" y="39.2176" smashed="yes" rot="R90">
 <attribute name="NAME" x="31.0896" y="37.9476" size="0.6096" layer="25" rot="R90"/>
 <attribute name="VALUE" x="34.2646" y="37.9476" size="0.6096" layer="25" rot="R90"/>
@@
 <signal name="N$1">
 <contactref element="ARDUINO" pad="7"/>
-<contactref element="U$7" pad="2"/>
+<contactref element="XTAL" pad="2"/>
 <contactref element="C2" pad="2"/>
 <wire x1="30.3276" y1="41.0276" x2="31.7496" y2="41.0276" width="0.254" layer="16"/>
@@
 <signal name="N$2">
 <contactref element="ARDUINO" pad="8"/>
-<contactref element="U$7" pad="1"/>
+<contactref element="XTAL" pad="1"/>
 <contactref element="C1" pad="2"/>
 <wire x1="30.3276" y1="40.2276" x2="31.3496" y2="40.2276" width="0.254" layer="16"/>
