File: Hardware/MoodBadge.sch (EAGLE design)
At the start: 46 parts

Commit message: updates
Parts:
- renumbered U$7 to XTAL
Changed lines of the file:
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@@
 <part name="U$3" library="CalvEngIO-Symbols" deviceset="VLIPO" device=""/>
 <part name="U$4" library="CalvEngIO-Symbols" deviceset="VLIPO" device=""/>
-<part name="U$7" library="OrlandoRonMod" deviceset="CRYSTAL-CA-310" device=""/>
+<part name="XTAL" library="OrlandoRonMod" deviceset="CRYSTAL-CA-310" device=""/>
 <part name="C1" library="CalvEngIO-Passives" deviceset="CAPACITOR" device="0402" value="22p"/>
 <part name="C2" library="CalvEngIO-Passives" deviceset="CAPACITOR" device="0402" value="22p"/>
@@
 <instance part="U$3" gate="G$1" x="53.34" y="218.44"/>
 <instance part="U$4" gate="G$1" x="45.72" y="238.76"/>
-<instance part="U$7" gate="G$1" x="55.88" y="198.12" rot="R90"/>
+<instance part="XTAL" gate="G$1" x="55.88" y="198.12" rot="R90"/>
 <instance part="C1" gate="G$1" x="55.88" y="190.5" rot="R180"/>
 <instance part="C2" gate="G$1" x="45.72" y="190.5" rot="R180"/>
@@
 <segment>
 <pinref part="ARDUINO" gate="G$1" pin="PB6(XTAL1/TOSC1)"/>
-<pinref part="U$7" gate="G$1" pin="2"/>
+<pinref part="XTAL" gate="G$1" pin="2"/>
 <wire x1="58.42" y1="200.66" x2="55.88" y2="200.66" width="0.1524" layer="91"/>
 <pinref part="C2" gate="G$1" pin="2"/>
@@
 <segment>
 <pinref part="ARDUINO" gate="G$1" pin="PB7(XTAL2/TOSC2)"/>
-<pinref part="U$7" gate="G$1" pin="1"/>
+<pinref part="XTAL" gate="G$1" pin="1"/>
 <wire x1="58.42" y1="195.58" x2="55.88" y2="195.58" width="0.1524" layer="91"/>
 <pinref part="C1" gate="G$1" pin="2"/>
